File: P6/P6.kicad_pcb (KiCad board)
At the start: 2 copper layers, 25 parts, among them J1 Conn_01x10, J2 Conn_01x10, SW13 SW_SPST, SW14 SW_SPST, SW15 SW_SPST, SW16 SW_SPST

Commit message: Finish PS6
Parts:
- moved D2 11.5 mm to (124.2, 266.2), turned to 180 degrees
- moved D1 11.5 mm to (60.2, 266.2), turned to 180 degrees
- moved SW14 11.5 mm to (124.2, 202.2), turned to 270 degrees
- moved SW13 11.5 mm to (60.2, 202.2), turned to 270 degrees
- moved D3 11.2 mm to (186.9, 266.2), turned to 180 degrees
- moved D4 11.2 mm to (250.9, 266.2), turned to 180 degrees
- moved SW15 11.2 mm to (186.9, 202.2), turned to 270 degrees
- moved SW16 11.2 mm to (250.9, 202.2), turned to 270 degrees
- moved C1 10.2 mm to (221.0, 35.6)
- moved C2 10.2 mm to (88.9, 35.6)
- moved H1 10.2 mm to (88.9, 61.0)
- moved H2 10.2 mm to (221.0, 60.9)
- moved J1 10.2 mm to (195.3, 29.0)
- moved J2 10.2 mm to (131.8, 29.0)
- moved H3 10.2 mm to (88.9, 200.7)
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Routing:
- net +15V: track 484.4 -> 898.7 mm
- net /6_LED2: track 0.00 -> 389.8 mm
- net GND: track 141.9 -> 518.3 mm
- net /5_LED1: track 0.00 -> 358.2 mm
- net /2_LED3: track 0.00 -> 336.9 mm
- net /3_LED4: track 0.00 -> 310.7 mm
- net /15_SW13: track 0.00 -> 240.0 mm
- net /11_SW16: track 0.00 -> 236.2 mm
- net Net-(D1-Pad2): track 0.00 -> 209.8 mm
- net /12_SW15: track 0.00 -> 197.9 mm
- net /14_SW14: track 0.00 -> 195.3 mm
Other:
- board outline added: 228.6 x 254 mm
