File: P6/P6.kicad_pcb (KiCad board)
At the start: 2 copper layers, 228.6 x 254 mm, 25 parts, among them J1 Conn_01x10, J2 Conn_01x10, SW13 SW_SPST, SW14 SW_SPST, SW15 SW_SPST, SW16 SW_SPST

Commit message: Update P6 to KiCad 7
Parts:
- moved ZD1 59.0 mm to (96.8, 210.3)
- moved D1 56.7 mm to (103.4, 229.4)
- moved SW13 48.7 mm to (101.6, 176.6)
- moved D2 46.9 mm to (152.9, 229.1)
- moved RV25 45.5 mm to (106.9, 89.2)
- moved H3 43.4 mm to (126.7, 179.3)
- moved RV26 43.4 mm to (107.4, 140.5)
- moved H1 41.6 mm to (127.0, 77.7)
- moved D3 40.8 mm to (202.2, 228.3)
- moved J2 40.7 mm to (162.8, 55.4)
- moved C2 38.8 mm to (121.7, 56.4)
- moved D4 37.8 mm to (251.7, 228.3)
- moved SW14 37.7 mm to (151.4, 176.1)
- moved RV27 32.0 mm to (156.4, 88.9)
- moved J1 30.4 mm to (212.1, 54.4)
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Routing:
- net +15V: track 898.7 -> 774.6 mm, vias 0 -> 4
- net -15V: track 542.5 -> 467.8 mm, vias 0 -> 4
- net /5_LED1: track 358.2 -> 301.4 mm
- net /3_LED4: track 310.7 -> 256.2 mm
- net /12_SW15: track 197.9 -> 145.7 mm
- net /15_SW13: track 240.0 -> 188.5 mm
- net /14_SW14: track 195.3 -> 145.5 mm
- net /2_LED3: track 336.9 -> 287.5 mm
- net /6_LED2: track 389.8 -> 341.8 mm
- net /11_SW16: track 236.2 -> 188.7 mm
- net /16_RV28: track 151.7 -> 113.6 mm
- net Net-(D1-A): track 209.8 -> 172.1 mm
- net GND: track 518.3 -> 481.8 mm, vias 0 -> 2
- net /19_RV25: track 81.5 -> 54.5 mm
- net /18_RV26: track 148.8 -> 124.1 mm
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Other:
- board size 228.6 x 254 mm -> 180.8 x 191.8 mm
- net class Default removed
- net class Power removed
