File: P5/P5.kicad_pcb (KiCad board)
At the start: 2 copper layers, 500 x 310 mm, 122 parts, among them J1 Conn_01x10, J2 Conn_01x10, J3 Conn_01x10, J4 Conn_01x10, J5 Conn_01x05, Q1 BC1, SW1 SW_Rotary1x3, SW10 SW_SPDT, SW11 SW_SPDT, SW12 SW_SPST, SW2 SW_SPDT, SW3 SW_SPDT, SW4 SW_Rotary1x3, SW5 SW_Rotary1x3, SW6 SW_Rotary1x3, SW7 SW_SPDT, SW8 SW_SPDT, SW8B1 SW_SPDT, SW9 SW_SPST, U1 TL072, U2 TL072, U3 LM741, U4 TL072, U5 4070, U6 4006, U7 LM741

Commit message: Add PS6 board
Parts:
- moved C1 275.9 mm to (-330.7, 43.4)
- moved R5 267.8 mm to (-326.5, -56.4)
- moved R4 264.2 mm to (-315.7, 73.4)
- moved C2 239.3 mm to (-315.7, 43.4)
- moved C3 239.3 mm to (-300.7, 43.4)
- moved C4 239.3 mm to (-285.7, 43.4)
- moved C5 239.3 mm to (-270.7, 43.4)
- moved C6 239.3 mm to (-255.7, 43.4)
- moved C7 239.3 mm to (-240.7, 43.4)
- moved C10 236.7 mm to (-315.7, 58.4)
- moved C8 236.7 mm to (-330.7, 58.4)
- moved LED1 236.7 mm to (-300.7, 58.4)
- moved Q1 236.7 mm to (-270.7, 58.4)
- moved R1 236.7 mm to (-255.7, 58.4)
- moved R2 236.7 mm to (-240.7, 58.4)
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
Commit message: Place components on P5, add front panel
Parts:
- moved R38_1 785.9 mm to (467.4, 299.7), turned to 90 degrees
- moved R37 732.0 mm to (401.3, 137.2), turned to 90 degrees
- moved PR1 698.8 mm to (408.9, 134.6), turned to 90 degrees
- moved R25 697.5 mm to (370.8, 292.1), turned to 90 degrees
- moved R26 687.7 mm to (378.5, 281.9), turned to 270 degrees
- moved ZD1 686.0 mm to (414.0, 190.5), turned to 180 degrees
- moved R38 684.5 mm to (365.8, 198.1), turned to 180 degrees
- moved R23 672.1 mm to (332.7, 210.8), turned to 90 degrees
- moved C3 671.2 mm to (348.0, 215.9), turned to 180 degrees
- moved U4 668.5 mm to (350.5, 203.2), turned to 270 degrees
- moved C10 656.4 mm to (325.1, 200.7)
- moved R24 653.6 mm to (332.7, 185.4), turned to 90 degrees
- moved SW8B1 650.4 mm to (378.5, 172.7)
- moved U3 645.7 mm to (315.0, 139.7), turned to 270 degrees
- moved R11 642.5 mm to (266.7, 119.4), turned to 90 degrees
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
Commit message: Fix P5 VCA/VCF A/D/R pots orientation
Parts:
- moved C1 16.2 mm to (232.4, 163.8)
- moved C10 16.2 mm to (336.6, 212.1)
- moved C2 16.2 mm to (295.9, 163.8)
- moved C3 16.2 mm to (359.4, 227.3)
- moved C4 16.2 mm to (268.0, 278.1)
- moved C6 16.2 mm to (242.6, 285.8)
- moved C8 16.2 mm to (196.8, 298.4)
- moved LED1 16.2 mm to (292.4, 301.0)
- moved PR1 16.2 mm to (420.4, 146.1)
- moved Q1 16.2 mm to (204.5, 280.7)
- moved R1 16.2 mm to (222.2, 163.8)
- moved R11 16.2 mm to (278.1, 130.8)
- moved R15 16.2 mm to (331.5, 166.4)
- moved R18 16.2 mm to (225.8, 80.5)
- moved R19 16.2 mm to (177.0, 225.2)
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Connections:
- net /35_DIG_0V renamed GNDD
- C7 pad 2: -15V -> GND
- J1 pad 1: /1_-15V -> -15V
- J1 pad 4: /4_+15V -> +15V
- J2 pad 5: (no net) -> -15V
- J2 pad 7: (no net) -> GND
- J4 pad 2: (no net) -> +15V
- J4 pad 3: (no net) -> -15V
- R25 pad 1: /4_+15V -> Net-(R25-Pad1)
- R26 pad 1: /1_-15V -> Net-(R26-Pad1)
- RV12 pad 1: GND -> -15V
- RV12 pad 3: -15V -> GND
- RV14 pad 1: GND -> -15V
- RV14 pad 3: -15V -> GND
- RV18 pad 1: GND -> -15V
- RV18 pad 3: -15V -> GND
- RV21 pad 1: GND -> -15V
- RV21 pad 3: -15V -> GND
- RV22 pad 1: GND -> -15V
- RV22 pad 3: -15V -> GND
- RV24 pad 1: GND -> -15V
- RV24 pad 3: -15V -> GND
- U1 pad 4: -15V -> Net-(R26-Pad1)
- U1 pad 8: +15V -> Net-(R25-Pad1)
- U2 pad 4: -15V -> Net-(R26-Pad1)
- U2 pad 8: +15V -> Net-(R25-Pad1)
- U4 pad 4: -15V -> Net-(R26-Pad1)
- U4 pad 8: +15V -> Net-(R25-Pad1)
- U5 pad 7: -15V -> GND

Commit message: P5 layout in progress
Parts:
- moved R42 23.9 mm to (76.2, 127.0), turned to 180 degrees
- moved R48 23.7 mm to (76.2, 191.5), turned to 180 degrees
- moved PR3 22.4 mm to (147.3, 237.5), turned to 270 degrees
- moved R44 22.0 mm to (76.2, 106.7), turned to 180 degrees
- moved R47 21.6 mm to (66.0, 196.6)
- moved R50 21.4 mm to (76.2, 171.1), turned to 180 degrees
- moved R41 21.2 mm to (66.0, 132.1)
- moved R45 19.1 mm to (66.0, 111.8)
- moved R51 19.1 mm to (66.0, 176.2)
- moved R40 16.8 mm to (52.1, 243.8), turned to 270 degrees
- moved R13 15.6 mm to (114.3, 142.2), turned to 180 degrees
- moved PR2 12.3 mm to (158.8, 222.2), turned to 90 degrees
- moved R43 11.4 mm to (76.2, 116.8), turned to 180 degrees
- moved R38_1 10.5 mm to (481.3, 301.0), turned to 270 degrees
- moved R27 10.2 mm to (288.3, 293.4), turned to 0 degrees
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Connections:
- RV13 pad 1: +15V -> -15V
- RV13 pad 3: -15V -> +15V
- SW1 pad 1: /36_VOICE4 -> /38_VOICE1
- SW1 pad 3: /38_VOICE1 -> /36_VOICE4
Routing:
- net -15V: track 0.00 -> 1153.8 mm
- net +15V: track 0.00 -> 1060.6 mm
- net GND: track 0.00 -> 990.5 mm
- net /39_VCO2_SAW: track 0.00 -> 515.8 mm
- net /40_VCO2_TRI: track 0.00 -> 500.2 mm
- net /41_VCO2_SQR: track 0.00 -> 470.9 mm
- net /42_VCO1_SAW: track 0.00 -> 422.7 mm
- net /27_VCO2_PWM_MOD: track 0.00 -> 418.3 mm
- net /43_VCO1_TRI: track 0.00 -> 407.1 mm
- net /44_VCO1_SQR: track 0.00 -> 391.6 mm
- net /28_VCO1_PWM_MOD: track 0.00 -> 358.3 mm
- net /3_ADSR_CONT_VCA: track 0.00 -> 306.6 mm
- net /26_VCO1_VOL: track 0.00 -> 305.2 mm
- net /45_PORTAMENTO: track 0.00 -> 295.6 mm
- net /2_ADSR_TRACK_VCA: track 0.00 -> 282.5 mm
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Other:
- net class Default: trace_width 0.25 -> 0.5
