File: P5/P5.sch (KiCad schematic (older format))
At the start: 122 parts, among them J1 Conn_01x10, J2 Conn_01x10, J3 Conn_01x10, J4 Conn_01x10, J5 Conn_01x05, Q1 BC1, SW1 SW_Rotary1x3, SW10 SW_SPDT, SW11 SW_SPDT, SW12 SW_SPST, SW2 SW_SPDT, SW3 SW_SPDT, SW4 SW_Rotary1x3, SW5 SW_Rotary1x3, SW6 SW_Rotary1x3, SW7 SW_SPDT, SW8 SW_SPDT, SW8B1 SW_SPDT, SW9 SW_SPST, U1 TL072, U2 TL072, U3 LM741, U4 TL072, U5 4070, U6 4006, U7 LM741

Commit message: Update PS3 & PS5
Parts:
- removed RV10, RV2: 22k, symbol Device:R_POT_MountingPin
- added RV10, RV2: 22k, P5:Potentiometer_Omeg_PC16BU_Vertical_Tapped, symbol P5:R_POT_US_TAPPED
- C1, C2, C3, C4, C5, C6, C7, C8: footprint (none) -> Capacitor_THT:C_Rect_L7.0mm_W3.5mm_P2.50mm_P5.00mm
- C10, C9: footprint (none) -> Capacitor_THT:CP_Radial_D5.0mm_P2.50mm
- J1, J2, J3, J4: footprint (none) -> Connector_PinHeader_2.54mm:PinHeader_1x10_P2.54mm_Vertical
- J5: footprint (none) -> Connector_PinHeader_2.54mm:PinHeader_1x05_P2.54mm_Vertical
- LED1: footprint (none) -> LED_THT:LED_D3.0mm
- PR1, PR2, PR3: footprint (none) -> Potentiometer_THT:Potentiometer_Bourns_3296W_Vertical
- Q1: footprint (none) -> Package_TO_SOT_THT:TO-92L_Wide
- R1, R10, R11, R12, R13, R14, R15, R16, R17, R18, R19, R2, R20, R21, R22, R23, R24, R25, R26, R27, R28, R29, R3, R30, R31, R32, R33, R34, R35, R36, R37, R38, R38_1, R39, R4, R40, R41, R42, R43, R44, R45, R46, R47, R48, R49, R5, R50, R51, R52, R53, R53_1, R6, R7, R8, R9: footprint (none) -> Resistor_THT:R_Axial_DIN0207_L6.3mm_D2.5mm_P10.16mm_Horizontal
- RV1, RV11, RV12, RV13, RV14, RV15, RV16, RV17, RV18, RV19, RV20, RV21, RV22, RV23, RV24, RV3, RV5, RV6, RV7, RV8, RV9: footprint (none) -> Potentiometer_THT:Potentiometer_Omeg_PC16BU_Vertical
- RV4: footprint (none) -> P5:Potentiometer_Omeg_PC16BU_Vertical_Tapped; symbol Device:R_POT_MountingPin -> P5:R_POT_US_TAPPED
- SW1, SW4, SW5, SW6: footprint (none) -> P5:SR2612F-0304-18R0B-D8-N
- SW10, SW11, SW12, SW7, SW8, SW8B1, SW9: footprint (none) -> P5:11-SS-22-701C
- SW2, SW3: footprint (none) -> Button_Switch_THT:SW_NKK_G1xJP
- U1, U2, U3, U4, U7: footprint (none) -> Package_DIP:DIP-8_W7.62mm_LongPads
- U5: footprint (none) -> Package_DIP:DIP-14_W7.62mm_LongPads
- U6: footprint (none) -> Package_DIP:DIP-14_W7.62mm_LongPads; symbol 4xxx_IEEE:4006 -> P5:4006
- ZD1: footprint (none) -> Diode_THT:D_A-405_P10.16mm_Horizontal
Connections:
- net Vdd is gone; now on net +15V: U6.14 (VDD)
- net Vss is gone; now on net GND: U6.7 (GND)
- net +15V: now also RV10.1
- net -15V: now also RV10.3
- net 30_VCF_ADSR_SWEEP: now also RV10.2
- net GND: now also RV4.4, RV10.4, RV2.4; no longer RV4.MP (MountPin)
- net at R15.2, RV4.1, U3.6: now also RV2.1
- net at R13.2: now also RV2.2
- net at R12.1: now also RV2.3
Other:
- moved on the sheet: C7, R33

Commit message: Fix P5 VCA/VCF A/D/R pots orientation
Connections:
- net 15_-15V is gone; now on net -15V: J2.5 (Pin_5)
- net 17_GND is gone; now on net GND: J2.7 (Pin_7)
- net 32_+15V is gone; now on net +15V: J4.2 (Pin_2)
- net 33_-15V is gone; now on net -15V: J4.3 (Pin_3)
- net 35_DIG_0V is gone; now on net GNDD: J4.5 (Pin_5), SW1.4, SW2.2 (B)
- net +15V: now also J1.4 (Pin_4); no longer U1.8 (V+), U2.8 (V+), U4.8 (V+)
- net -15V: now also J1.1 (Pin_1), RV12.1, RV14.1, RV18.1, RV21.1, RV22.1, RV24.1; no longer C7.2, RV12.3, RV14.3, RV18.3, RV21.3, RV22.3, RV24.3, U1.4 (V-), U2.4 (V-), U4.4 (V-), U5.7 (VSS)
- net GND: now also C7.2, RV12.3, RV14.3, RV18.3, RV21.3, RV22.3, RV24.3, U5.7 (VSS); no longer RV12.1, RV14.1, RV18.1, RV21.1, RV22.1, RV24.1
- net 1_-15V: no longer names the net of R26.1
- net 1_-15V: now also U1.4 (V-), U2.4 (V-), U4.4 (V-); no longer J1.1 (Pin_1)
- net 4_+15V: no longer names the net of R25.1
- net 4_+15V: now also U1.8 (V+), U2.8 (V+), U4.8 (V+); no longer J1.4 (Pin_4)
- no-connect marks 14 -> 10
Other:
- moved on the sheet: C10, C9, R25, R26, U1C, U2C, U4C, U5E

Commit message: P5 layout in progress
Connections:
- net +15V: now also RV13.3; no longer RV13.1
- net -15V: now also RV13.1; no longer RV13.3
- net 36_VOICE4: now also SW1.3; no longer SW1.1
- net 38_VOICE1: now also SW1.1; no longer SW1.3
Changed lines of the file:
@@
 F 3 "~" H 14850 4900 50  0001 C CNN
 	1    14850 4900
-	1    0    0    -1
+	1    0    0    1
 $EndComp
 Wire Wire Line
@@
 F 3 "http://cdn-reichelt.de/documents/datenblatt/C200/DS-Serie%23LOR.pdf" H 10750 1350 50  0001 C CNN
 	1    10850 1050
-	-1   0    0    -1
-$EndComp
-$Comp
+	-1   0    0    1
+$EndComp
+$Comp
