File: P3/P3.sch (KiCad schematic (older format))
At the start: 96 parts, among them J1 Conn_01x10, J2 Conn_01x05, J3 Conn_01x10, J4 Conn_01x05, J5 Conn_02x07_Counter_Clockwise, U1 SN75107B, U10 74LS08, U11 7425, U12 74LS32, U13 74LS193, U14 74LS153, U15 74LS74, U16 74LS93, U17 74LS244, U18 74LS367, U19 74LS367, U2 74LS175, U20 74LS32, U21 74LS74, U22 74LS266, U23 74LS266, U24 6810-Memory_RAM-eti-polysynth, U25 74LS08, U26 74LS08, U27 CD4051B, U28 74LS259, U29 74LS13, U3 74LS74, U30 74LS93, U31 74LS93, U32 74LS93, U33 74LS42, U34 74LS32, U35 74LS04, U36 7404, U37 4041, U38 4041, U39 TL072, U4 D2102, U40 TL082, U41 TL082, U42 TL082, U43 TL082, U44 L7805, U5 74LS00, U6 74LS04, U7 74LS10, U8 74LS00, U9 74LS32

Commit message: Update PS3 & PS5
Parts:
- added C14, C15, C16, C17, C18, C19, C20, C21, C22, C23: 10uF, Capacitor_THT:CP_Radial_D8.0mm_P5.00mm, symbol Device:CP_Small
- added H1, H2, H3, H4, H5, H6, H7, H8: MountingHole, MountingHole:MountingHole_3.2mm_M3_DIN965_Pad, symbol Mechanical:MountingHole
- added HS1: Heatsink, Heatsink:Heatsink_Fischer_SK129-STS_42x25mm_2xDrill2.5mm, symbol Mechanical:Heatsink
- added J6: Screw_Terminal_01x02, TerminalBlock:TerminalBlock_Altech_AK300-2_P5.00mm, symbol Connector:Screw_Terminal_01x02
- added unit 5 of U22
- added unit 5 of U23
- U16: footprint Package_DIP:DIP-10_W7.62mm_LongPads -> Package_DIP:DIP-14_W7.62mm_LongPads
- renumbered D4 to D3, D3 to D4
Connections:
- net -15V is gone; now on net -5V: U39.4 (V-), U40.4 (V-), U41.4 (V-), U42.4 (V-), U43.4 (V-)
- net +5V: now also C14.1, C15.1, C16.1, C17.1, C18.1, C19.1, C20.1, C21.1, C22.1, C23.1, U22.14 (VCC), U23.14 (VCC)
- net D4: now also U38.13 (D)
- net D5: now also U38.10 (C)
- net GND: now also D1.2 (A), D2.2 (A), C14.2, C15.2, C16.2, C17.2, C18.2, C19.2, C20.2, C21.2, C22.2, C23.2, U22.7 (GND), U23.7 (GND); no longer D2.1 (K), D3.2 (A)
- net P3: now also U41.1, U41.2 (-); no longer U41.6 (-), U41.7
- net P4: now also U41.6 (-), U41.7; no longer U41.1, U41.2 (-)
- net P5: now also U42.1, U42.2 (-); no longer U42.6 (-), U42.7
- net P6: now also U43.6 (-), U43.7; no longer U42.1, U42.2 (-)
- net P7: now also U42.6 (-), U42.7; no longer U43.6 (-), U43.7
- net at C5.1, U27.1 (X4): now also U42.3 (+); no longer U42.5 (+)
- net at C4.1, U27.12 (X3): now also U41.5 (+); no longer U41.3 (+)
- net at C3.1, U27.15 (X2): now also U41.3 (+); no longer U41.5 (+)
- net at C7.1, U27.2 (X6): now also U42.5 (+); no longer U43.5 (+)
- net at C6.1, U27.5 (X5): now also U43.5 (+); no longer U42.3 (+)
- net at R21.2, U38.1 (A): now also U38.11 (D)
- net at R23.2, U38.4 (B): now also U38.8 (C)
- net at C12.1, C9.1, U44.1 (IN): now also D3.1 (K), D4.1 (K); no longer D1.1 (K), D4.2 (A)
- removed net AC: D1.2 (A), D2.2 (A), D3.1 (K), D4.1 (K)
- new net: D1.1 (K), D4.2 (A), J6.1 (Pin_1)
- new net: D2.1 (K), D3.2 (A), J6.2 (Pin_2)
- no-connect marks 96 -> 92
Other:
- moved on the sheet: C12, C13, C9, D1, D2, D3, D4, J1, J2, J3, J4, R21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

Commit message: P3 layout in progress
Parts:
- C12, C13, C14, C15, C16, C17, C18, C19, C20, C21, C22, C23, C24, C25, C26, C27: footprint Capacitor_THT:CP_Radial_D8.0mm_P5.00mm -> Capacitor_THT:CP_Radial_D6.3mm_P2.50mm
- J5: symbol Connector_Generic:Conn_02x07_Counter_Clockwise -> Connector_Generic:Conn_02x07_Odd_Even
- U22, U23: footprint (none) -> Package_DIP:DIP-14_W7.62mm_LongPads
Connections:
- net +5V: now also J5.4 (Pin_4), J5.7 (Pin_7); no longer J5.1 (Pin_1), J5.11 (Pin_11)
- net -5V: now also J5.6 (Pin_6), J5.8 (Pin_8); no longer J5.3 (Pin_3), J5.4 (Pin_4)
- net A0: now also U4.2 (A5); no longer U4.8 (A0)
- net A5: now also U4.8 (A0); no longer U4.2 (A5)
- net FROM_KEYBOARD: now also J5.5 (Pin_5); no longer J5.12 (Pin_12)
- net GND: now also J5.1 (Pin_1), J5.3 (Pin_3); no longer J5.13 (Pin_13), J5.14 (Pin_14)
- net K0: now also J5.14 (Pin_14); no longer J5.7 (Pin_7)
- net K1: now also J5.12 (Pin_12); no longer J5.6 (Pin_6)
- net K2: now also J5.10 (Pin_10); no longer J5.5 (Pin_5)
- net K3: now also J5.13 (Pin_13); no longer J5.8 (Pin_8)
- net K4: now also J5.11 (Pin_11); no longer J5.9 (Pin_9)
- net K5: now also J5.9 (Pin_9); no longer J5.10 (Pin_10)
- net at U8.11: now also U10.4; no longer U10.5
- net at U7.8: now also U10.5; no longer U10.4
- net U17_0EA: now reaches U17.1 (OEa)
- net U17_0EA: now also U20.11; no longer U20.3
- net U17_0EB: now reaches U17.19 (OEb)
- net U17_0EB: now also U20.3; no longer U20.11
- net ~RW renamed R~W
Other:
- note added: "Master Clock/Timing Generator"
- moved on the sheet: U20A, U20D

Commit message: P3 layout in progress 2
Connections:
- net ~CP2: now also U34.9; no longer U34.10
- net at U29.8, U34.2, U35.9: now also U34.10; no longer U34.9
Changed lines of the file:
@@
 U 3 1 5E8A6081
 P 5850 12400
-F 0 "U34" H 5850 12725 50  0000 C CNN
-F 1 "74LS32" H 5850 12634 50  0000 C CNN
+F 0 "U34" H 5850 12050 50  0000 C CNN
+F 1 "74LS32" H 5850 12150 50  0000 C CNN
 F 2 "Package_DIP:DIP-14_W7.62mm_LongPads" H 5850 12400 50  0001 C CNN
 F 3 "http://www.ti.com/lit/gpn/sn74LS32" H 5850 12400 50  0001 C CNN
 	3    5850 12400
-	1    0    0    -1
+	1    0    0    1
 $EndComp
 Text Label 11100 13150 2    50   ~ 0
