File: P3/P3.kicad_pcb (KiCad board)
At the start: 2 copper layers, 116 parts, among them J1 Conn_01x10, J2 Conn_01x05, J3 Conn_01x10, J4 Conn_01x05, J5 Conn_02x07_Counter_Clockwise, J6 Screw_Terminal_01x02, U1 SN75107B, U10 74LS08, U11 7425, U12 74LS32, U13 74LS193, U14 74LS153, U15 74LS74, U16 74LS93, U17 74LS244, U18 74LS367, U19 74LS367, U2 74LS175, U20 74LS32, U21 74LS74, U22 74LS266, U23 74LS266, U24 6810-Memory_RAM-eti-polysynth, U25 74LS08, U26 74LS08, U27 CD4051B, U28 74LS259, U29 74LS13, U3 74LS74, U30 74LS93, U31 74LS93, U32 74LS93, U33 74LS42, U34 74LS32, U35 74LS04, U36 7404, U37 4041, U38 4041, U39 TL072, U4 D2102, U40 TL082, U41 TL082, U42 TL082, U43 TL082, U44 L7805, U5 74LS00, U6 74LS04, U7 74LS10, U8 74LS00, U9 74LS32

Commit message: P3 layout in progress
Parts:
- C12, C13, C14, C15, C16, C17, C18, C19, C20, C21, C22, C23, C24, C25, C26, C27: footprint Capacitor_THT:CP_Radial_D8.0mm_P5.00mm -> Capacitor_THT:CP_Radial_D6.3mm_P2.50mm
- moved R4 12.2 mm to (208.5, 134.6), turned to 270 degrees
- moved H3 11.5 mm to (116.1, 25.3)
- moved H5 11.4 mm to (224.1, 25.4)
- moved C15 10.7 mm to (54.9, 127.0), turned to 180 degrees
- moved C14 9.14 mm to (29.0, 76.2)
- moved C19 9.03 mm to (176.8, 119.6), turned to 270 degrees
- moved C24 8.74 mm to (206.4, 150.7)
- moved R1 7.37 mm to (197.9, 130.3), turned to 180 degrees
- moved C11 5.23 mm to (91.0, 132.0), turned to 270 degrees
- moved C10 5.08 mm to (101.6, 67.3), turned to 270 degrees
- moved C17 4.20 mm to (107.5, 128.3)
- moved C18 4.10 mm to (142.2, 128.2)
- moved U4 2.54 mm to (163.8, 104.1)
- moved C21 2.53 mm to (231.2, 154.3), turned to 90 degrees
- moved R2 2.03 mm to (218.2, 144.8)
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Connections:
- net /~RW renamed /R~W
- J5 pad 1: +5V -> GND
- J5 pad 10: /K5 -> /K2
- J5 pad 11: +5V -> /K4
- J5 pad 12: /FROM_KEYBOARD -> /K1
- J5 pad 13: GND -> /K3
- J5 pad 14: GND -> /K0
- J5 pad 3: -5V -> GND
- J5 pad 4: -5V -> +5V
- J5 pad 5: /K2 -> /FROM_KEYBOARD
- J5 pad 6: /K1 -> -5V
- J5 pad 7: /K0 -> +5V
- J5 pad 8: /K3 -> -5V
- J5 pad 9: /K4 -> /K5
- U17 pad 1: Net-(U17-Pad1) -> /U17_0EA
- U17 pad 19: Net-(U17-Pad19) -> /U17_0EB
- U20 pad 11: Net-(U17-Pad19) -> /U17_0EA
- U20 pad 3: Net-(U17-Pad1) -> /U17_0EB
- U4 pad 2: /A5 -> /A0
- U4 pad 8: /A0 -> /A5
- U7 pad 8: Net-(U10-Pad4) -> Net-(U10-Pad5)
- U8 pad 11: Net-(U10-Pad5) -> Net-(U10-Pad4)
Routing:
- net GND: track 590.2 -> 1292.0 mm
- net /~CLC: track 0.00 -> 601.9 mm, vias 0 -> 4
- net +5V: track 1226.2 -> 1719.4 mm
- net /~ANC: track 0.00 -> 474.2 mm, vias 0 -> 4
- net Net-(U18-Pad11): track 0.00 -> 439.5 mm, vias 0 -> 6
- net /SL1: track 0.00 -> 423.7 mm, vias 0 -> 4
- net /SL2: track 0.00 -> 411.6 mm, vias 0 -> 4
- net /MODE_SWITCH: track 0.00 -> 365.4 mm
- net Net-(U27-Pad6): track 0.00 -> 364.9 mm, vias 0 -> 4
- net /~CP1: track 8.67 -> 359.2 mm
- net /CLC: track 0.00 -> 340.2 mm, vias 0 -> 2
- net /~CP2: track 0.00 -> 325.5 mm, vias 0 -> 4
- net /IC2_11: track 0.00 -> 314.6 mm, vias 0 -> 2
- net /~KU: track 0.00 -> 287.7 mm, vias 0 -> 4
- net /R~W: track 0.00 -> 270.3 mm, vias 0 -> 7
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
Commit message: P3 layout in progress 2
Parts:
- moved H4 2.67 mm to (138.4, 183.1)
- moved H6 1.84 mm to (255.8, 183.5)
Connections:
- U34 pad 10: /~CP2 -> Net-(U29-Pad8)
- U34 pad 9: Net-(U29-Pad8) -> /~CP2
Routing:
- net Net-(U29-Pad8): track 0.00 -> 224.8 mm, vias 0 -> 4
- net /IC18_7: track 253.8 -> 454.1 mm, vias 3 -> 6
- net /A2: track 213.5 -> 405.8 mm, vias 4 -> 7
- net /IC18_5: track 271.7 -> 457.0 mm, vias 3 -> 6
- net /IC18_3: track 240.0 -> 408.8 mm, vias 5 -> 8
- net /F2: track 12.3 -> 119.5 mm, vias 0 -> 6
- net Net-(U4-Pad11): track 0.00 -> 89.4 mm, vias 0 -> 2
- net /F0: track 0.00 -> 85.8 mm, vias 0 -> 4
- net /F1: track 22.8 -> 105.8 mm, vias 0 -> 4
- net /IC2-D3: track 0.00 -> 73.2 mm, vias 0 -> 2
- net Net-(U12-Pad12): track 0.00 -> 72.8 mm
- net +5V: track 1719.4 -> 1654.1 mm
- net /IC14_5: track 0.00 -> 61.3 mm, vias 0 -> 2
- net /IC2-D2: track 0.00 -> 60.6 mm
- net /~TGU: track 32.3 -> 87.8 mm, vias 0 -> 2
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
Commit message: P3 layout in progress 2
Parts:
- moved C12 41.7 mm to (310.2, 95.8)
- moved C13 41.7 mm to (323.9, 95.8)
- moved C27 41.7 mm to (348.0, 212.9)
- moved R17 40.5 mm to (322.0, 176.7)
- moved U39 40.5 mm to (336.4, 196.3)
- moved H4 40.5 mm to (149.9, 222.0)
- moved R12 40.5 mm to (322.0, 160.8)
- moved U28 40.5 mm to (367.3, 138.4)
- moved C19 40.5 mm to (188.3, 158.4)
- moved C24 40.5 mm to (217.9, 189.5)
- moved D1 40.5 mm to (346.0, 87.9)
- moved D2 40.5 mm to (351.3, 87.9)
- moved R22 40.5 mm to (311.8, 192.5)
- moved U18 40.5 mm to (201.3, 89.7)
- moved U34 40.5 mm to (144.1, 170.9)
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Routing:
- net GND: track 1291.4 -> 1377.0 mm
- net Net-(U11-Pad5): track 34.5 -> 80.6 mm
- net Net-(U11-Pad4): track 43.0 -> 85.2 mm
- net Net-(U11-Pad2): track 37.2 -> 64.2 mm
- net Net-(U11-Pad1): track 43.1 -> 62.3 mm
- net +15V: track 178.5 -> 166.9 mm
- net /~CLC: track 601.9 -> 591.3 mm
- net /IC2_11: track 313.1 -> 303.3 mm
- net /SL2: track 411.6 -> 402.4 mm
- net /SL1: track 423.7 -> 414.7 mm
- net /CLC: track 340.2 -> 332.0 mm
- net /4_VOICE: track 179.7 -> 185.2 mm
- net /MODE_SWITCH: track 365.4 -> 359.9 mm
- net /A2: track 405.8 -> 401.1 mm
- net +5V: track 1654.1 -> 1658.5 mm
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Other:
- board text added: "DGND"
