File: P3/P3.kicad_sch (KiCad schematic)
At the start: 116 parts, among them J1 Conn_01x10, J2 Conn_01x05, J3 Conn_01x10, J4 Conn_01x05, J5 Conn_02x07_Counter_Clockwise, J6 Screw_Terminal_01x02, U1 SN75107B, U10 74LS08, U11 7425, U12 74LS32, U13 74LS193, U14 74LS153, U15 74LS74, U16 74LS93, U17 74LS244, U18 74LS367, U19 74LS367, U2 74LS175, U20 74LS32, U21 74LS74, U22 74LS266, U23 74LS266, U24 6810-Memory_RAM-eti-polysynth, U25 74LS08, U26 74LS08, U27 CD4051B, U28 74LS259, U29 74LS13, U3 74LS74, U30 74LS93, U31 74LS93, U32 74LS93, U33 74LS42, U34 74LS32, U35 74LS04, U36 7404, U37 4041, U38 4041, U39 TL072, U4 D2102, U40 TL082, U41 TL082, U42 TL082, U43 TL082, U44 L7805, U5 74LS00, U6 74LS04, U7 74LS10, U8 74LS00, U9 74LS32

Commit message: Update P3 to KiCad 7
Parts:
- C12, C13, C14, C15, C16, C17, C18, C19, C20, C21, C22, C23, C24, C25, C26, C27, C9: symbol P3-rescue:CP_Small-Device -> Device:C_Polarized_Small
- U24: footprint Package_DIP:DIP-24_W15.24mm_LongPads -> Package_DIP:DIP-24_W10.16mm_LongPads
