File: P4/P4.kicad_pcb (KiCad board)
At the start: 2 copper layers, 126 parts, among them J1 Conn_01x10, J11 Conn_01x10, J12 Conn_01x10, J13 Conn_01x25, J14 Conn_01x25, J15 Conn_01x25, J16 Conn_01x25, J17 Conn_01x25, J18 Conn_01x25, J19 Conn_01x25, J2 Conn_01x10, J20 Conn_01x25, J26 Conn_01x01, J3 Conn_01x10, J4 Conn_01x10, J5 Conn_01x05, J6 Conn_01x10, J7 Conn_01x10, J8 Conn_01x03, J9 Conn_01x03, Q1 BC212L, Q2 BC212L, Q3 TIP42, Q4 TIP41, U1 LM723_DIP14, U10 LM13600, U11 LF353, U12 LM741, U13 LM13600, U2 LM741, U3 L7905, U4 LM1458, U5 LM1458, U6 LF353, U7 LM13600, U8 LF353, U9 LF353

Commit message: Update PS4 board/schematic
Parts:
- added J21: Conn_01x25, Connector_PinSocket_2.54mm:PinSocket_1x25_P2.54mm_Vertical, F.Cu at (276.9, 167.6)
- added J22: Conn_01x25, Connector_PinSocket_2.54mm:PinSocket_1x25_P2.54mm_Vertical, F.Cu at (276.9, 101.6)
- moved RA39 110.6 mm to (162.1, 150.6), turned to 270 degrees
- moved RB40 100.0 mm to (165.4, 158.2), turned to 90 degrees
- moved CA21 93.8 mm to (158.8, 150.6), turned to 270 degrees
- moved RB31 74.0 mm to (79.2, 157.2), turned to 0 degrees
- moved CB20 73.2 mm to (144.8, 157.2), turned to 180 degrees
- moved RA30 72.1 mm to (77.0, 157.2), turned to 180 degrees
- moved CA15 68.8 mm to (77.0, 153.9), turned to 180 degrees
- moved CB22 64.7 mm to (145.3, 174.5), turned to 180 degrees
- moved RC41 62.5 mm to (139.7, 150.6)
- moved RC38 61.5 mm to (139.7, 153.9)
- moved CB16 46.8 mm to (94.2, 157.2), turned to 180 degrees
- moved RC35 42.1 mm to (89.2, 150.6)
- moved RC32 40.5 mm to (89.2, 153.9)
- moved CB18 38.1 mm to (94.5, 174.5), turned to 180 degrees
- moved RA36 30.9 mm to (127.5, 157.2), turned to 180 degrees
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Connections:
- net /U1_PIN10 renamed Net-(Q4-Pad1)
Routing:
- net GND: track 870.4 -> 1261.7 mm, vias 0 -> 6
- net -15V: track 453.9 -> 709.3 mm
- net -5V: track 143.9 -> 353.4 mm, vias 0 -> 2
- net +15V: track 435.2 -> 609.3 mm
- net /35_VOICE1_OUT: track 98.7 -> 264.1 mm, vias 0 -> 1
- net /3_VOICE_1_PITCH: track 0.00 -> 158.7 mm, vias 0 -> 2
- net /P4: track 0.00 -> 156.5 mm, vias 0 -> 1
- net /3_VOICE_3_PITCH: track 0.00 -> 143.0 mm, vias 0 -> 2
- net /P3: track 0.00 -> 128.0 mm, vias 0 -> 1
- net /3_VOICE_2_PITCH: track 0.00 -> 120.3 mm, vias 0 -> 2
- net /P2: track 0.00 -> 116.2 mm, vias 0 -> 1
- net /3_VOICE_4_PITCH: track 0.00 -> 114.7 mm, vias 0 -> 2
- net /P1: track 0.00 -> 67.8 mm
- net /VOICE1_PORTAMENTO: track 0.00 -> 59.6 mm
- net Net-(CA17-Pad1): track 0.00 -> 48.8 mm
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Other:
- board outline added: 267.2 x 216.4 mm

Commit message: P4 layout in progress
Parts:
- moved R2 48.2 mm to (121.8, 127.4)
- moved R10 47.8 mm to (116.3, 123.8)
- moved R9 47.8 mm to (119.9, 123.8)
- moved R8 47.0 mm to (121.8, 112.6)
- moved C1 45.7 mm to (107.1, 127.4)
- moved U5 44.0 mm to (108.4, 116.2)
- moved C4 42.3 mm to (107.1, 112.6)
- moved R1 42.1 mm to (95.6, 126.9)
- moved R4 42.1 mm to (95.6, 123.8)
- moved R6 42.1 mm to (95.6, 116.2)
- moved R7 42.1 mm to (95.6, 113.2)
- moved C2 39.5 mm to (79.8, 127.4)
- moved U4 38.3 mm to (81.1, 116.2)
- moved C3 37.1 mm to (79.8, 112.6)
- moved R3 34.4 mm to (67.1, 127.4)
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Connections:
- R3 pad 2: /42_G3 -> /42_G2
- R5 pad 2: /42_G2 -> /42_G3
- U11 pad 2: /3_VOICE_4_PITCH -> /3_VOICE_1_PITCH
- U11 pad 3: /P4 -> /P1
- U11 pad 6: /3_VOICE_4_PITCH -> /3_VOICE_1_PITCH
- U11 pad 7: /3_VOICE_4_PITCH -> /3_VOICE_1_PITCH
- U6 pad 2: /3_VOICE_1_PITCH -> /3_VOICE_4_PITCH
- U6 pad 3: /P1 -> /P4
- U6 pad 6: /3_VOICE_1_PITCH -> /3_VOICE_4_PITCH
- U6 pad 7: /3_VOICE_1_PITCH -> /3_VOICE_4_PITCH
- U8 pad 2: /3_VOICE_2_PITCH -> /3_VOICE_3_PITCH
- U8 pad 3: /P2 -> /P3
- U8 pad 6: /3_VOICE_2_PITCH -> /3_VOICE_3_PITCH
- U8 pad 7: /3_VOICE_2_PITCH -> /3_VOICE_3_PITCH
- U9 pad 2: /3_VOICE_3_PITCH -> /3_VOICE_2_PITCH
- U9 pad 3: /P3 -> /P2
- U9 pad 6: /3_VOICE_3_PITCH -> /3_VOICE_2_PITCH
- U9 pad 7: /3_VOICE_3_PITCH -> /3_VOICE_2_PITCH
Routing:
- net GND: track 1261.7 -> 734.3 mm
- net +15V: track 609.3 -> 285.6 mm
- net -15V: track 709.3 -> 436.5 mm
- net -5V: track 353.4 -> 108.7 mm, vias 2 -> 1
- net /29_MASTER_VOLUME: track 51.9 -> 242.5 mm, vias 1 -> 2
- net /P4: track 156.5 -> 0.00 mm, vias 1 -> 0
- net /45_PORTAMENTO: track 0.00 -> 134.9 mm, vias 0 -> 2
- net /P3: track 128.0 -> 0.00 mm, vias 1 -> 0
- net /-: track 117.8 -> 0.00 mm
- net /P2: track 116.2 -> 0.00 mm, vias 1 -> 0
- net /3_VOICE_4_PITCH: track 114.7 -> 229.4 mm
- net /3_VOICE_1_PITCH: track 158.7 -> 47.8 mm, vias 2 -> 0
- net /+: track 76.6 -> 0.00 mm
- net /P1: track 67.8 -> 0.00 mm
- net Net-(R10-Pad2): track 60.2 -> 0.00 mm
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Other:
- board size 267.2 x 216.4 mm -> 267.2 x 184.3 mm

Commit message: P4 layout in progress
Parts:
- moved CB18 1.57 mm to (76.2, 157.5)
- moved CB22 1.57 mm to (127.0, 157.5)
- moved R22 0.64 mm to (101.2, 163.1)
- moved C12 0.57 mm to (96.1, 163.0)
Routing:
- net /P1: track 0.00 -> 142.1 mm, vias 0 -> 1
- net GND: track 734.3 -> 876.1 mm
- net /VOICE1_PORTAMENTO: track 4.99 -> 126.0 mm, vias 0 -> 2
- net +15V: track 285.6 -> 399.0 mm, vias 0 -> 4
- net /P2: track 0.00 -> 107.0 mm, vias 0 -> 1
- net /1_PITCH_BEND: track 137.8 -> 235.1 mm, vias 1 -> 2
- net /P3: track 0.00 -> 90.2 mm, vias 0 -> 1
- net -15V: track 436.5 -> 525.6 mm, vias 0 -> 2
- net Net-(CA17-Pad1): track 0.00 -> 48.3 mm
- net Net-(CA21-Pad1): track 0.00 -> 46.8 mm
- net /P4: track 0.00 -> 43.7 mm
- net Net-(CB20-Pad2): track 0.00 -> 41.5 mm
- net Net-(CB16-Pad2): track 0.00 -> 41.0 mm
- net Net-(RC35-Pad2): track 0.00 -> 26.9 mm
- net Net-(CB22-Pad2): track 0.00 -> 25.1 mm
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
Commit message: P4 layout in progress
Parts:
- moved R42 12.9 mm to (30.2, 69.1), turned to 270 degrees
- moved J8 5.08 mm to (132.3, 74.7)
- moved C11 4.70 mm to (39.6, 71.1)
- moved C9 4.25 mm to (81.0, 79.9)
- moved R16 2.95 mm to (42.2, 79.2)
- moved C7 1.82 mm to (91.1, 79.9), turned to 180 degrees
- moved R14 1.03 mm to (76.3, 84.3)
- moved R12 0.89 mm to (106.9, 78.8)
- moved U1 0.51 mm to (109.5, 84.3)
- moved ZD1 0.32 mm to (63.6, 79.9)
Routing:
- net GND: track 876.1 -> 994.9 mm
- net /-: track 0.00 -> 107.9 mm
- net Net-(R10-Pad2): track 0.00 -> 84.2 mm
- net /+: track 0.00 -> 66.4 mm
- net +15V: track 399.0 -> 456.9 mm
- net /2_L3: track 0.00 -> 54.5 mm, vias 0 -> 1
- net /6_L2: track 0.00 -> 50.7 mm, vias 0 -> 1
- net /42_G1: track 395.3 -> 445.6 mm, vias 2 -> 3
- net Net-(C8-Pad1): track 0.00 -> 49.9 mm
- net Net-(Q3-Pad3): track 0.00 -> 43.2 mm
- net Net-(R13-Pad2): track 0.00 -> 40.2 mm
- net -15V: track 525.6 -> 557.1 mm
- net Net-(D1-Pad1): track 0.00 -> 22.7 mm
- net Net-(D2-Pad1): track 0.00 -> 21.0 mm
- net /5_L1: track 0.00 -> 16.1 mm, vias 0 -> 1
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
Commit message: P4 layout in progress
Parts:
- moved R17 2.54 mm to (53.5, 72.6)
- moved RB40 1.40 mm to (148.6, 142.6)
- moved CA15 1.40 mm to (60.2, 138.3)
- moved CA17 1.40 mm to (90.2, 134.5)
- moved CA19 1.40 mm to (110.7, 138.3)
- moved CA21 1.40 mm to (142.0, 135.0)
- moved CB16 1.40 mm to (77.5, 141.6)
- moved CB20 1.40 mm to (128.0, 141.6)
- moved RA30 1.40 mm to (60.2, 141.6)
- moved RA33 1.40 mm to (94.5, 134.5)
- moved RA36 1.40 mm to (110.7, 141.6)
- moved RA39 1.40 mm to (145.3, 135.0)
- moved RB31 1.40 mm to (62.5, 141.6)
- moved RB34 1.40 mm to (97.8, 142.1)
- moved RB37 1.40 mm to (113.0, 141.6)
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Routing:
- net -5V: track 114.6 -> 345.7 mm, vias 1 -> 4
- net GND: track 994.9 -> 1135.2 mm
- net +15V: track 456.9 -> 547.3 mm
- net -15V: track 557.1 -> 638.1 mm
- net Net-(Q2-Pad3): track 0.00 -> 44.7 mm, vias 0 -> 2
- net Net-(Q4-Pad1): track 0.00 -> 33.0 mm, vias 0 -> 2
- net /35_VOICE1_OUT: track 263.2 -> 248.3 mm
- net /11_ADSR4_ON_OFF: track 94.9 -> 108.7 mm
- net Net-(R15-Pad1): track 0.00 -> 13.3 mm
- net Net-(Q2-Pad2): track 0.00 -> 9.66 mm
- net /12_ADSR3_ON_OFF: track 69.4 -> 76.1 mm, vias 1 -> 2
- net Net-(U2-Pad7): track 0.00 -> 6.45 mm
- net Net-(Q1-Pad2): track 9.18 -> 15.4 mm
- net Net-(Q3-Pad3): track 43.2 -> 40.8 mm
- net /P1: track 142.1 -> 139.8 mm
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