File: P1-2/P1-2.kicad_sch (KiCad schematic)
At the start: 83 parts, among them J1 Conn_02x07_Odd_Even, Q1 BC212L, SW1 Conn_01x01_Pin, SW10 Conn_01x01_Pin, SW11 Conn_01x01_Pin, SW12 Conn_01x01_Pin, SW13 Conn_01x01_Pin, SW14 Conn_01x01_Pin, SW15 Conn_01x01_Pin, SW16 Conn_01x01_Pin, SW17 Conn_01x01_Pin, SW18 Conn_01x01_Pin, SW19 Conn_01x01_Pin, SW2 Conn_01x01_Pin, SW20 Conn_01x01_Pin, SW21 Conn_01x01_Pin, SW22 Conn_01x01_Pin, SW23 Conn_01x01_Pin, SW24 Conn_01x01_Pin, SW25 Conn_01x01_Pin, SW26 Conn_01x01_Pin, SW27 Conn_01x01_Pin, SW28 Conn_01x01_Pin, SW29 Conn_01x01_Pin, SW3 Conn_01x01_Pin, SW30 Conn_01x01_Pin, SW31 Conn_01x01_Pin, SW32 Conn_01x01_Pin, SW33 Conn_01x01_Pin, SW34 Conn_01x01_Pin, SW35 Conn_01x01_Pin, SW36 Conn_01x01_Pin, SW37 Conn_01x01_Pin, SW38 Conn_01x01_Pin, SW39 Conn_01x01_Pin, SW4 Conn_01x01_Pin, SW40 Conn_01x01_Pin, SW41 Conn_01x01_Pin, SW42 Conn_01x01_Pin, SW43 Conn_01x01_Pin, SW44 Conn_01x01_Pin, SW45 Conn_01x01_Pin, SW46 Conn_01x01_Pin, SW47 Conn_01x01_Pin, SW48 Conn_01x01_Pin, SW49 Conn_01x01_Pin, SW5 Conn_01x01_Pin, SW6 Conn_01x01_Pin, SW7 Conn_01x01_Pin, SW8 Conn_01x01_Pin, SW9 Conn_01x01_Pin, U1 4051, U2 4051, U3 4051, U4 4051, U5 4051, U6 4051, U7 4051, U8 74LS42

Commit message: Finish P1-2
Parts:
- added J2, J3: Conn_01x11_Pin, Connector_PinHeader_2.54mm:PinHeader_1x11_P2.54mm_Vertical, symbol Connector:Conn_01x11_Pin
Connections:
- net +5V: now also J2.11 (Pin_11), J3.11 (Pin_11)
- net -5V: now also J2.10 (Pin_10), J3.10 (Pin_10)
- net 3: now also J2.9 (Pin_9), J3.9 (Pin_9)
- net 4: now also J2.8 (Pin_8), J3.8 (Pin_8)
- net 5: now also J2.7 (Pin_7), J3.7 (Pin_7)
- net 6: now also J2.6 (Pin_6), J3.6 (Pin_6)
- net A0: now also J2.3 (Pin_3), J3.3 (Pin_3)
- net A1: now also J2.4 (Pin_4), J3.4 (Pin_4)
- net A2: now also J2.5 (Pin_5), J3.5 (Pin_5)
- net GND: now also C4.2, C5.1, J2.1 (Pin_1), J3.1 (Pin_1)
- net KEYSCAN_OUT: now reaches R3.2, U1.3 (X), U2.3 (X), U3.3 (X), U4.3 (X), U5.3 (X), U6.3 (X), U7.3 (X)
- net KEYSCAN_OUT: now also J2.2 (Pin_2), J3.2 (Pin_2)
Other:
- moved on the sheet: C4, C5
