File: P1-2/P1-2.kicad_sch (KiCad schematic)
At the start: 85 parts, among them J1 Conn_02x07_Odd_Even, J2 Conn_01x11_Pin, J3 Conn_01x11_Pin, Q1 BC212L, SW1 Conn_01x01_Pin, SW10 Conn_01x01_Pin, SW11 Conn_01x01_Pin, SW12 Conn_01x01_Pin, SW13 Conn_01x01_Pin, SW14 Conn_01x01_Pin, SW15 Conn_01x01_Pin, SW16 Conn_01x01_Pin, SW17 Conn_01x01_Pin, SW18 Conn_01x01_Pin, SW19 Conn_01x01_Pin, SW2 Conn_01x01_Pin, SW20 Conn_01x01_Pin, SW21 Conn_01x01_Pin, SW22 Conn_01x01_Pin, SW23 Conn_01x01_Pin, SW24 Conn_01x01_Pin, SW25 Conn_01x01_Pin, SW26 Conn_01x01_Pin, SW27 Conn_01x01_Pin, SW28 Conn_01x01_Pin, SW29 Conn_01x01_Pin, SW3 Conn_01x01_Pin, SW30 Conn_01x01_Pin, SW31 Conn_01x01_Pin, SW32 Conn_01x01_Pin, SW33 Conn_01x01_Pin, SW34 Conn_01x01_Pin, SW35 Conn_01x01_Pin, SW36 Conn_01x01_Pin, SW37 Conn_01x01_Pin, SW38 Conn_01x01_Pin, SW39 Conn_01x01_Pin, SW4 Conn_01x01_Pin, SW40 Conn_01x01_Pin, SW41 Conn_01x01_Pin, SW42 Conn_01x01_Pin, SW43 Conn_01x01_Pin, SW44 Conn_01x01_Pin, SW45 Conn_01x01_Pin, SW46 Conn_01x01_Pin, SW47 Conn_01x01_Pin, SW48 Conn_01x01_Pin, SW49 Conn_01x01_Pin, SW5 Conn_01x01_Pin, SW6 Conn_01x01_Pin, SW7 Conn_01x01_Pin, SW8 Conn_01x01_Pin, SW9 Conn_01x01_Pin, U1 4051, U2 4051, U3 4051, U4 4051, U5 4051, U6 4051, U7 4051, U8 74LS42

Commit message: Update P1-2 and ignore backups
Parts:
- added H1, H2, H3, H4, H5, H6: MountingHole, MountingHole:MountingHole_3mm_Pad, symbol Mechanical:MountingHole
Changed lines of the file:
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@@
   (junction (at 251.46 24.13) (diameter 0) (color 0 0 0 0)
   )
+  (junction (at 100.33 36.83) (diameter 0) (color 0 0 0 0)
+  )
   (junction (at 374.65 121.92) (diameter 0) (color 0 0 0 0)
   )
@@
     (stroke (width 0) (type default))
   )
+  (wire (pts (xy 100.33 36.83) (xy 102.87 36.83))
+    (stroke (width 0) (type default))
+  )
   (wire (pts (xy 242.57 81.28) (xy 294.64 81.28))
     (stroke (width 0) (type default))
@@
     (stroke (width 0) (type default))
   )
-  (wire (pts (xy 83.82 36.83) (xy 102.87 36.83))
+  (wire (pts (xy 83.82 36.83) (xy 100.33 36.83))
     (stroke (width 0) (type default))
   )
@@
       (effects (font (size 1.27 1.27)) (justify right))
     )
-    (property "Footprint" "Diode_THT:D_DO-35_SOD27_P7.62mm_Horizontal" (at 302.895 43.18 0)
+    (property "Footprint" "Diode_THT:D_DO-35_SOD27_P7.62mm_Horizontal" (at 307.34 43.18 0)
       (effects (font (size 1.27 1.27)) hide)
     )
@@
       (effects (font (size 1.27 1.27)) hide)
     )
+    (property "Sim.Device" "D" (at 307.34 43.18 0)
+      (effects (font (size 1.27 1.27)) hide)
+    )
+    (property "Sim.Pins" "1=K 2=A" (at 307.34 43.18 0)
+      (effects (font (size 1.27 1.27)) hide)
+    )
     (pin "1")
     (pin "2")
@@
     )
   )
+  (symbol (lib_id "Mechanical:MountingHole") (at 120.015 48.895 0) (unit 1)
+    (in_bom yes) (on_board yes) (dnp no) (fields_autoplaced)
+    (property "Reference" "H3" (at 123.19 47.625 0)
+      (effects (font (size 1.27 1.27)) (justify left))
+    )
+    (property "Value" "MountingHole" (at 123.19 50.165 0)
+      (effects (font (size 1.27 1.27)) (justify left))
+    )
+    (property "Footprint" "MountingHole:MountingHole_3mm_Pad" (at 120.015 48.895 0)
+      (effects (font (size 1.27 1.27)) hide)
+    )
+    (property "Datasheet" "~" (at 120.015 48.895 0)
+      (effects (font (size 1.27 1.27)) hide)
+    )
+    (instances
+      (project "P1-2"
+        (path "/63ae384a-573f-42cb-925b-0486f86a73c0"
+          (reference "H3") (unit 1)
+        )
+      )
+    )
+  )
   (symbol (lib_id "Connector:Conn_01x11_Pin") (at 281.94 185.42 0) (unit 1)
     (in_bom yes) (on_board yes) (dnp no)
@@
     )
   )
+  (symbol (lib_id "Mechanical:MountingHole") (at 140.335 33.655 0) (unit 1)
+    (in_bom yes) (on_board yes) (dnp no) (fields_autoplaced)
+    (property "Reference" "H4" (at 143.51 32.385 0)
+      (effects (font (size 1.27 1.27)) (justify left))
+    )
+    (property "Value" "MountingHole" (at 143.51 34.925 0)
+      (effects (font (size 1.27 1.27)) (justify left))
+    )
+    (property "Footprint" "MountingHole:MountingHole_3mm_Pad" (at 140.335 33.655 0)
+      (effects (font (size 1.27 1.27)) hide)
+    )
+    (property "Datasheet" "~" (at 140.335 33.655 0)
+      (effects (font (size 1.27 1.27)) hide)
+    )
+    (instances
+      (project "P1-2"
+        (path "/63ae384a-573f-42cb-925b-0486f86a73c0"
+          (reference "H4") (unit 1)
+        )
+      )
+    )
+  )
+  (symbol (lib_id "Mechanical:MountingHole") (at 120.015 33.655 0) (unit 1)
+    (in_bom yes) (on_board yes) (dnp no) (fields_autoplaced)
+    (property "Reference" "H1" (at 123.19 32.385 0)
+      (effects (font (size 1.27 1.27)) (justify left))
+    )
+    (property "Value" "MountingHole" (at 123.19 34.925 0)
+      (effects (font (size 1.27 1.27)) (justify left))
+    )
+    (property "Footprint" "MountingHole:MountingHole_3mm_Pad" (at 120.015 33.655 0)
+      (effects (font (size 1.27 1.27)) hide)
+    )
+    (property "Datasheet" "~" (at 120.015 33.655 0)
+      (effects (font (size 1.27 1.27)) hide)
+    )
+    (instances
+      (project "P1-2"
+        (path "/63ae384a-573f-42cb-925b-0486f86a73c0"
+          (reference "H1") (unit 1)
+        )
+      )
+    )
+  )
+  (symbol (lib_id "power:PWR_FLAG") (at 100.33 36.83 0) (unit 1)
+    (in_bom yes) (on_board yes) (dnp no)
+    (property "Reference" "#FLG01" (at 100.33 34.925 0)
+      (effects (font (size 1.27 1.27)) hide)
+    )
+    (property "Value" "PWR_FLAG" (at 100.33 31.75 0)
+      (effects (font (size 1.27 1.27)))
+    )
+    (property "Footprint" "" (at 100.33 36.83 0)
+      (effects (font (size 1.27 1.27)) hide)
+    )
+    (property "Datasheet" "~" (at 100.33 36.83 0)
+      (effects (font (size 1.27 1.27)) hide)
+    )
+    (pin "1")
+    (instances
+      (project "P1-2"
+        (path "/63ae384a-573f-42cb-925b-0486f86a73c0"
+          (reference "#FLG01") (unit 1)
+        )
+      )
+    )
+  )
+  (symbol (lib_id "Mechanical:MountingHole") (at 120.015 41.275 0) (unit 1)
+    (in_bom yes) (on_board yes) (dnp no) (fields_autoplaced)
+    (property "Reference" "H2" (at 123.19 40.005 0)
+      (effects (font (size 1.27 1.27)) (justify left))
+    )
+    (property "Value" "MountingHole" (at 123.19 42.545 0)
+      (effects (font (size 1.27 1.27)) (justify left))
+    )
+    (property "Footprint" "MountingHole:MountingHole_3mm_Pad" (at 120.015 41.275 0)
+      (effects (font (size 1.27 1.27)) hide)
+    )
+    (property "Datasheet" "~" (at 120.015 41.275 0)
+      (effects (font (size 1.27 1.27)) hide)
+    )
+    (instances
+      (project "P1-2"
+        (path "/63ae384a-573f-42cb-925b-0486f86a73c0"
+          (reference "H2") (unit 1)
+        )
+      )
+    )
+  )
   (symbol (lib_id "power:+5V") (at 255.27 204.47 0) (unit 1)
     (in_bom yes) (on_board yes) (dnp no)
@@
         )
       )
+    )
+  )
+  (symbol (lib_id "Mechanical:MountingHole") (at 140.335 48.895 0) (unit 1)
+    (in_bom yes) (on_board yes) (dnp no) (fields_autoplaced)
+    (property "Reference" "H6" (at 143.51 47.625 0)
+      (effects (font (size 1.27 1.27)) (justify left))
+    )
+    (property "Value" "MountingHole" (at 143.51 50.165 0)
+      (effects (font (size 1.27 1.27)) (justify left))
+    )
+    (property "Footprint" "MountingHole:MountingHole_3mm_Pad" (at 140.335 48.895 0)
+      (effects (font (size 1.27 1.27)) hide)
+    )
+    (property "Datasheet" "~" (at 140.335 48.895 0)
+      (effects (font (size 1.27 1.27)) hide)
+    )
+    (instances
+      (project "P1-2"
+        (path "/63ae384a-573f-42cb-925b-0486f86a73c0"
+          (reference "H6") (unit 1)
+        )
+      )
+    )
+  )
+  (symbol (lib_id "Mechanical:MountingHole") (at 140.335 41.275 0) (unit 1)
+    (in_bom yes) (on_board yes) (dnp no) (fields_autoplaced)
+    (property "Reference" "H5" (at 143.51 40.005 0)
+      (effects (font (size 1.27 1.27)) (justify left))
+    )
+    (property "Value" "MountingHole" (at 143.51 42.545 0)
+      (effects (font (size 1.27 1.27)) (justify left))
+    )
+    (property "Footprint" "MountingHole:MountingHole_3mm_Pad" (at 140.335 41.275 0)
+      (effects (font (size 1.27 1.27)) hide)
+    )
+    (property "Datasheet" "~" (at 140.335 41.275 0)
+      (effects (font (size 1.27 1.27)) hide)
+    )
+    (instances
+      (project "P1-2"
+        (path "/63ae384a-573f-42cb-925b-0486f86a73c0"
+          (reference "H5") (unit 1)
+        )
+      )
