File: P1-2/P1-2.kicad_pcb (KiCad board)
At the start: 2 copper layers, 688.3 x 86.4 mm, 85 parts, among them J1 Conn_02x07_Odd_Even, J2 Conn_01x11_Pin, J3 Conn_01x11_Pin, Q1 BC212L, SW1 Conn_01x01_Pin, SW10 Conn_01x01_Pin, SW11 Conn_01x01_Pin, SW12 Conn_01x01_Pin, SW13 Conn_01x01_Pin, SW14 Conn_01x01_Pin, SW15 Conn_01x01_Pin, SW16 Conn_01x01_Pin, SW17 Conn_01x01_Pin, SW18 Conn_01x01_Pin, SW19 Conn_01x01_Pin, SW2 Conn_01x01_Pin, SW20 Conn_01x01_Pin, SW21 Conn_01x01_Pin, SW22 Conn_01x01_Pin, SW23 Conn_01x01_Pin, SW24 Conn_01x01_Pin, SW25 Conn_01x01_Pin, SW26 Conn_01x01_Pin, SW27 Conn_01x01_Pin, SW28 Conn_01x01_Pin, SW29 Conn_01x01_Pin, SW3 Conn_01x01_Pin, SW30 Conn_01x01_Pin, SW31 Conn_01x01_Pin, SW32 Conn_01x01_Pin, SW33 Conn_01x01_Pin, SW34 Conn_01x01_Pin, SW35 Conn_01x01_Pin, SW36 Conn_01x01_Pin, SW37 Conn_01x01_Pin, SW38 Conn_01x01_Pin, SW39 Conn_01x01_Pin, SW4 Conn_01x01_Pin, SW40 Conn_01x01_Pin, SW41 Conn_01x01_Pin, SW42 Conn_01x01_Pin, SW43 Conn_01x01_Pin, SW44 Conn_01x01_Pin, SW45 Conn_01x01_Pin, SW46 Conn_01x01_Pin, SW47 Conn_01x01_Pin, SW48 Conn_01x01_Pin, SW49 Conn_01x01_Pin, SW5 Conn_01x01_Pin, SW6 Conn_01x01_Pin, SW7 Conn_01x01_Pin, SW8 Conn_01x01_Pin, SW9 Conn_01x01_Pin, U1 4051, U2 4051, U3 4051, U4 4051, U5 4051, U6 4051, U7 4051, U8 74LS42

Commit message: Update P1-2 and ignore backups
Parts:
- added H1: MountingHole, MountingHole:MountingHole_3mm_Pad, F.Cu at (97.0, 67.3)
- added H2: MountingHole, MountingHole:MountingHole_3mm_Pad, F.Cu at (249.9, 67.3)
- added H3: MountingHole, MountingHole:MountingHole_3mm_Pad, F.Cu at (402.3, 67.3)
- added H4: MountingHole, MountingHole:MountingHole_3mm_Pad, F.Cu at (436.4, 67.3)
- added H5: MountingHole, MountingHole:MountingHole_3mm_Pad, F.Cu at (603.8, 67.3)
- added H6: MountingHole, MountingHole:MountingHole_3mm_Pad, F.Cu at (756.7, 67.3)
Changed lines of the file:
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@@
     )
   )
+  (footprint "MountingHole:MountingHole_3mm_Pad" (layer "F.Cu")
+    (at 97.028 67.31)
+    (descr "Mounting Hole 3mm")
+    (tags "mounting hole 3mm")
+    (property "Sheetfile" "P1-2.kicad_sch")
+    (property "Sheetname" "")
+    (property "ki_description" "Mounting Hole without connection")
+    (property "ki_keywords" "mounting hole")
+    (attr exclude_from_pos_files)
+    (fp_text reference "H1" (at 0 -4) (layer "F.SilkS")
+        (effects (font (size 1 1) (thickness 0.15)))
+    )
+    (fp_text value "MountingHole" (at 0 4) (layer "F.Fab")
+        (effects (font (size 1 1) (thickness 0.15)))
+    )
+    (fp_text user "${REFERENCE}" (at 0 0) (layer "F.Fab")
+        (effects (font (size 1 1) (thickness 0.15)))
+    )
+    (fp_circle (center 0 0) (end 3 0)
+      (stroke (width 0.15) (type solid)) (fill none) (layer "Cmts.User"))
+    (fp_circle (center 0 0) (end 3.25 0)
+      (stroke (width 0.05) (type solid)) (fill none) (layer "F.CrtYd"))
+    (pad "1" thru_hole circle (at 0 0) (size 6 6) (drill 3) (layers "*.Cu" "*.Mask"))
+  )
   (footprint "Connector_Pin:Pin_D1.3mm_L11.0mm_LooseFit" (layer "F.Cu")
     (at 486.791 92.456)
@@
     )
   )
+  (footprint "MountingHole:MountingHole_3mm_Pad" (layer "F.Cu")
+    (at 249.936 67.31)
+    (descr "Mounting Hole 3mm")
+    (tags "mounting hole 3mm")
+    (property "Sheetfile" "P1-2.kicad_sch")
+    (property "Sheetname" "")
+    (property "ki_description" "Mounting Hole without connection")
+    (property "ki_keywords" "mounting hole")
+    (attr exclude_from_pos_files)
+    (fp_text reference "H2" (at 0 -4) (layer "F.SilkS")
+        (effects (font (size 1 1) (thickness 0.15)))
+    )
+    (fp_text value "MountingHole" (at 0 4) (layer "F.Fab")
+        (effects (font (size 1 1) (thickness 0.15)))
+    )
+    (fp_text user "${REFERENCE}" (at 0 0) (layer "F.Fab")
+        (effects (font (size 1 1) (thickness 0.15)))
+    )
+    (fp_circle (center 0 0) (end 3 0)
+      (stroke (width 0.15) (type solid)) (fill none) (layer "Cmts.User"))
+    (fp_circle (center 0 0) (end 3.25 0)
+      (stroke (width 0.05) (type solid)) (fill none) (layer "F.CrtYd"))
+    (pad "1" thru_hole circle (at 0 0) (size 6 6) (drill 3) (layers "*.Cu" "*.Mask"))
+  )
   (footprint "Connector_Pin:Pin_D1.3mm_L11.0mm_LooseFit" (layer "F.Cu")
     (at 669.163 92.456)
@@
     (property "Sheetfile" "P1-2.kicad_sch")
     (property "Sheetname" "")
+    (property "Sim.Device" "D")
+    (property "Sim.Pins" "1=K 2=A")
     (property "ki_description" "100V 0.15A standard switching diode, DO-35")
     (property "ki_keywords" "diode")
@@
     )
   )
+  (footprint "MountingHole:MountingHole_3mm_Pad" (layer "F.Cu")
+    (at 402.336 67.31)
+    (descr "Mounting Hole 3mm")
+    (tags "mounting hole 3mm")
+    (property "Sheetfile" "P1-2.kicad_sch")
+    (property "Sheetname" "")
+    (property "ki_description" "Mounting Hole without connection")
+    (property "ki_keywords" "mounting hole")
+    (attr exclude_from_pos_files)
+    (fp_text reference "H3" (at 0 -4) (layer "F.SilkS")
+        (effects (font (size 1 1) (thickness 0.15)))
+    )
+    (fp_text value "MountingHole" (at 0 4) (layer "F.Fab")
+        (effects (font (size 1 1) (thickness 0.15)))
+    )
+    (fp_text user "${REFERENCE}" (at 0 0) (layer "F.Fab")
+        (effects (font (size 1 1) (thickness 0.15)))
+    )
+    (fp_circle (center 0 0) (end 3 0)
+      (stroke (width 0.15) (type solid)) (fill none) (layer "Cmts.User"))
+    (fp_circle (center 0 0) (end 3.25 0)
+      (stroke (width 0.05) (type solid)) (fill none) (layer "F.CrtYd"))
+    (pad "1" thru_hole circle (at 0 0) (size 6 6) (drill 3) (layers "*.Cu" "*.Mask"))
+  )
   (footprint "Capacitor_THT:CP_Radial_D5.0mm_P2.00mm" (layer "F.Cu")
     (at 503.555 108.712 90)
@@
     )
   )
+  (footprint "MountingHole:MountingHole_3mm_Pad" (layer "F.Cu")
+    (at 603.758 67.31)
+    (descr "Mounting Hole 3mm")
+    (tags "mounting hole 3mm")
+    (property "Sheetfile" "P1-2.kicad_sch")
+    (property "Sheetname" "")
+    (property "ki_description" "Mounting Hole without connection")
+    (property "ki_keywords" "mounting hole")
+    (attr exclude_from_pos_files)
+    (fp_text reference "H5" (at 0 -4) (layer "F.SilkS")
+        (effects (font (size 1 1) (thickness 0.15)))
+    )
+    (fp_text value "MountingHole" (at 0 4) (layer "F.Fab")
+        (effects (font (size 1 1) (thickness 0.15)))
+    )
+    (fp_text user "${REFERENCE}" (at 0 0) (layer "F.Fab")
+        (effects (font (size 1 1) (thickness 0.15)))
+    )
+    (fp_circle (center 0 0) (end 3 0)
+      (stroke (width 0.15) (type solid)) (fill none) (layer "Cmts.User"))
+    (fp_circle (center 0 0) (end 3.25 0)
+      (stroke (width 0.05) (type solid)) (fill none) (layer "F.CrtYd"))
+    (pad "1" thru_hole circle (at 0 0) (size 6 6) (drill 3) (layers "*.Cu" "*.Mask"))
+  )
   (footprint "Connector_Pin:Pin_D1.3mm_L11.0mm_LooseFit" (layer "F.Cu")
     (at 410.083 92.456)
@@
     )
   )
+  (footprint "MountingHole:MountingHole_3mm_Pad" (layer "F.Cu")
+    (at 436.372 67.31)
+    (descr "Mounting Hole 3mm")
+    (tags "mounting hole 3mm")
+    (property "Sheetfile" "P1-2.kicad_sch")
+    (property "Sheetname" "")
+    (property "ki_description" "Mounting Hole without connection")
+    (property "ki_keywords" "mounting hole")
+    (attr exclude_from_pos_files)
+    (fp_text reference "H4" (at 0 -4) (layer "F.SilkS")
+        (effects (font (size 1 1) (thickness 0.15)))
+    )
+    (fp_text value "MountingHole" (at 0 4) (layer "F.Fab")
+        (effects (font (size 1 1) (thickness 0.15)))
+    )
+    (fp_text user "${REFERENCE}" (at 0 0) (layer "F.Fab")
+        (effects (font (size 1 1) (thickness 0.15)))
+    )
+    (fp_circle (center 0 0) (end 3 0)
+      (stroke (width 0.15) (type solid)) (fill none) (layer "Cmts.User"))
+    (fp_circle (center 0 0) (end 3.25 0)
+      (stroke (width 0.05) (type solid)) (fill none) (layer "F.CrtYd"))
+    (pad "1" thru_hole circle (at 0 0) (size 6 6) (drill 3) (layers "*.Cu" "*.Mask"))
+  )
   (footprint "Connector_Pin:Pin_D1.3mm_L11.0mm_LooseFit" (layer "F.Cu")
     (at 457.835 92.456)
@@
     )
   )
+  (footprint "MountingHole:MountingHole_3mm_Pad" (layer "F.Cu")
+    (at 756.666 67.31)
+    (descr "Mounting Hole 3mm")
+    (tags "mounting hole 3mm")
+    (property "Sheetfile" "P1-2.kicad_sch")
+    (property "Sheetname" "")
+    (property "ki_description" "Mounting Hole without connection")
+    (property "ki_keywords" "mounting hole")
+    (attr exclude_from_pos_files)
+    (fp_text reference "H6" (at 0 -4) (layer "F.SilkS")
+        (effects (font (size 1 1) (thickness 0.15)))
+    )
+    (fp_text value "MountingHole" (at 0 4) (layer "F.Fab")
+        (effects (font (size 1 1) (thickness 0.15)))
+    )
+    (fp_text user "${REFERENCE}" (at 0 0) (layer "F.Fab")
+        (effects (font (size 1 1) (thickness 0.15)))
+    )
+    (fp_circle (center 0 0) (end 3 0)
+      (stroke (width 0.15) (type solid)) (fill none) (layer "Cmts.User"))
+    (fp_circle (center 0 0) (end 3.25 0)
+      (stroke (width 0.05) (type solid)) (fill none) (layer "F.CrtYd"))
+    (pad "1" thru_hole circle (at 0 0) (size 6 6) (drill 3) (layers "*.Cu" "*.Mask"))
+  )
   (footprint "Connector_Pin:Pin_D1.3mm_L11.0mm_LooseFit" (layer "F.Cu")
